File: MagicGlove/SkateMate_Glove.sch (EAGLE design)
At the start: 41 parts, among them U1 ATMEGA328P-AU, Y1 8MHz

Commit message: Version 0.1 Layout
Parts:
- removed POWERIN1: -, wirepad:1,6/0,8
- IC1: value (none) -> BU33TD3WG
Connections:
- net GND: no longer POWERIN1.P, Y1.1, Y1.2
- net N$3: now also Y1.1
- net N$4: now also Y1.2
Other:
- moved on the sheet: C4, C5
Changed lines of the file:
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@@
 <setting verticaltext="up"/>
 </settings>
-<grid distance="0.01" unitdist="inch" unit="inch" style="lines" multiple="1" display="no" altdistance="0.01" altunitdist="inch" altunit="inch"/>
+<grid distance="0.01" unitdist="inch" unit="mm" style="lines" multiple="1" display="no" altdistance="0.01" altunitdist="inch" altunit="mic"/>
 <layers>
 <layer number="1" name="Top" color="4" fill="1" visible="no" active="no"/>
@@
 <part name="PAD1" library="wirepad" deviceset="1,6/0,8" device="" value="-"/>
 <part name="PAD2" library="wirepad" deviceset="1,6/0,8" device="" value="+"/>
-<part name="IC1" library="BU33TD3WG" deviceset="BU33TD3WG-TR" device=""/>
+<part name="IC1" library="BU33TD3WG" deviceset="BU33TD3WG-TR" device="" value="BU33TD3WG"/>
 <part name="U$1" library="MCP73831" deviceset="MCP73831" device=""/>
 <part name="C7" library="eagle-ltspice" deviceset="C" device="C0603" value=".47u"/>
@@
 <part name="GND15" library="supply1" deviceset="GND" device=""/>
 <part name="POWERIN" library="wirepad" deviceset="1,6/0,8" device="" value="+"/>
-<part name="POWERIN1" library="wirepad" deviceset="1,6/0,8" device="" value="-"/>
-<part name="GND16" library="supply1" deviceset="GND" device=""/>
 </parts>
 <sheets>
@@
 <instance part="U1" gate="A" x="48.26" y="38.1"/>
 <instance part="C3" gate="G$1" x="15.24" y="63.5" rot="R90"/>
-<instance part="C4" gate="G$1" x="15.24" y="27.94" rot="R90"/>
-<instance part="C5" gate="G$1" x="15.24" y="17.78" rot="R90"/>
+<instance part="C4" gate="G$1" x="-3.302" y="27.94" rot="R90"/>
+<instance part="C5" gate="G$1" x="-3.556" y="17.78" rot="R90"/>
 <instance part="+3V34" gate="G$1" x="2.54" y="63.5" rot="R90"/>
 <instance part="GND4" gate="1" x="0" y="7.62"/>
 <instance part="Y1" gate="G$1" x="10.16" y="22.86" rot="R90"/>
-<instance part="GND3" gate="1" x="0" y="27.94" rot="R270"/>
+<instance part="GND3" gate="1" x="-12.7" y="23.876" rot="R270"/>
 <instance part="GND5" gate="1" x="-15.24" y="39.37" rot="R270"/>
 <instance part="C6" gate="G$1" x="-5.08" y="39.37" rot="R270"/>
@@
 <instance part="GND15" gate="1" x="59.436" y="-27.432"/>
 <instance part="POWERIN" gate="P" x="-31.496" y="2.032" rot="R270"/>
-<instance part="POWERIN1" gate="P" x="-41.402" y="2.286" rot="R270"/>
-<instance part="GND16" gate="1" x="-41.402" y="-8.636"/>
 </instances>
 <busses>
@@
 <wire x1="0" y1="15.24" x2="0" y2="12.7" width="0.1524" layer="91"/>
 <junction x="0" y="12.7"/>
-</segment>
-<segment>
-<pinref part="Y1" gate="G$1" pin="2"/>
-<pinref part="C4" gate="G$1" pin="1"/>
-<wire x1="10.16" y1="27.94" x2="12.7" y2="27.94" width="0.1524" layer="91"/>
-<pinref part="GND3" gate="1" pin="GND"/>
-<wire x1="2.54" y1="27.94" x2="10.16" y2="27.94" width="0.1524" layer="91"/>
-<junction x="10.16" y="27.94"/>
-<pinref part="Y1" gate="G$1" pin="1"/>
-<pinref part="C5" gate="G$1" pin="1"/>
-<wire x1="10.16" y1="17.78" x2="12.7" y2="17.78" width="0.1524" layer="91"/>
-<wire x1="10.16" y1="17.78" x2="2.54" y2="17.78" width="0.1524" layer="91"/>
-<wire x1="2.54" y1="17.78" x2="2.54" y2="27.94" width="0.1524" layer="91"/>
-<junction x="10.16" y="17.78"/>
-<junction x="2.54" y="27.94"/>
 </segment>
 <segment>
@@
 </segment>
 <segment>
-<pinref part="POWERIN1" gate="P" pin="P"/>
-<pinref part="GND16" gate="1" pin="GND"/>
-<wire x1="-41.402" y1="-0.254" x2="-41.402" y2="-6.096" width="0.1524" layer="91"/>
+<pinref part="C4" gate="G$1" pin="1"/>
+<pinref part="GND3" gate="1" pin="GND"/>
+<wire x1="-5.842" y1="27.94" x2="-10.16" y2="27.94" width="0.1524" layer="91"/>
+<wire x1="-10.16" y1="27.94" x2="-10.16" y2="23.876" width="0.1524" layer="91"/>
+<pinref part="C5" gate="G$1" pin="1"/>
+<wire x1="-6.096" y1="17.78" x2="-10.16" y2="17.78" width="0.1524" layer="91"/>
+<wire x1="-10.16" y1="17.78" x2="-10.16" y2="23.876" width="0.1524" layer="91"/>
+<junction x="-10.16" y="23.876"/>
 </segment>
 </net>
@@
 <pinref part="C7" gate="G$1" pin="1"/>
 <wire x1="136.652" y1="-23.876" x2="136.652" y2="-32.004" width="0.1524" layer="91"/>
-</segment>
-</net>
-<net name="N$3" class="0">
-<segment>
-<pinref part="U1" gate="A" pin="PB7"/>
-<pinref part="C5" gate="G$1" pin="2"/>
-<wire x1="20.32" y1="17.78" x2="20.32" y2="20.32" width="0.1524" layer="91"/>
-<wire x1="20.32" y1="20.32" x2="30.48" y2="20.32" width="0.1524" layer="91"/>
-</segment>
-</net>
-<net name="N$4" class="0">
-<segment>
-<pinref part="U1" gate="A" pin="PB6"/>
-<pinref part="C4" gate="G$1" pin="2"/>
-<wire x1="20.32" y1="27.94" x2="20.32" y2="22.86" width="0.1524" layer="91"/>
-<wire x1="20.32" y1="22.86" x2="30.48" y2="22.86" width="0.1524" layer="91"/>
+<junction x="136.652" y="-23.876"/>
 </segment>
 </net>
@@
 </segment>
 </net>
+<net name="N$3" class="0">
+<segment>
+<pinref part="U1" gate="A" pin="PB7"/>
+<wire x1="30.48" y1="20.32" x2="16.764" y2="20.32" width="0.1524" layer="91"/>
+<wire x1="16.764" y1="20.32" x2="16.764" y2="17.526" width="0.1524" layer="91"/>
+<pinref part="Y1" gate="G$1" pin="1"/>
+<wire x1="16.764" y1="17.526" x2="10.16" y2="17.526" width="0.1524" layer="91"/>
+<wire x1="10.16" y1="17.526" x2="10.16" y2="17.78" width="0.1524" layer="91"/>
+<pinref part="C5" gate="G$1" pin="2"/>
+<wire x1="10.16" y1="17.78" x2="1.524" y2="17.78" width="0.1524" layer="91"/>
+<junction x="10.16" y="17.78"/>
+</segment>
+</net>
+<net name="N$4" class="0">
+<segment>
+<pinref part="U1" gate="A" pin="PB6"/>
+<wire x1="30.48" y1="22.86" x2="16.764" y2="22.86" width="0.1524" layer="91"/>
+<wire x1="16.764" y1="22.86" x2="16.764" y2="27.94" width="0.1524" layer="91"/>
+<pinref part="Y1" gate="G$1" pin="2"/>
+<wire x1="16.764" y1="27.94" x2="10.16" y2="27.94" width="0.1524" layer="91"/>
+<pinref part="C4" gate="G$1" pin="2"/>
+<wire x1="10.16" y1="27.94" x2="1.778" y2="27.94" width="0.1524" layer="91"/>
+<junction x="10.16" y="27.94"/>
+</segment>
+</net>

Commit message: V0.9 Layout and Schematic ready for review and version jump to 1.0.
Parts:
- removed C10: 4.7u, eagle-ltspice:CC0603
- removed C4, C5: 22p, eagle-ltspice:CC0603
- removed POWERIN: +, wirepad:1,6/0,8
- removed SV2: RFM75, con-lstb:MA08-1
- removed Y1: 8MHz, crystals:ABM3
- added U$2: HEADER1,27, SkateMateMagicGlove:HEADER1,27
- added U$3: MICRO-USB-ZX62R-B-5P, con-hirose:MICRO-USB-ZX62R-B-5P
Connections:
- removed net N$3: C5.2, U1.PB7, Y1.1
- removed net N$4: C4.2, U1.PB6, Y1.2
- net +3V3: now also U$2.P$2; no longer SV2.2
- net CE: now also U$2.P$3; no longer SV2.3
- net CSN: now also U$2.P$4; no longer SV2.4
- net GND: now also U$2.P$1; no longer C10.2, C4.1, C5.1, SV2.1
- net IRQ: now also U$2.P$8; no longer SV2.8
- net MISO: now also U$2.P$7; no longer SV2.7
- net MOSI: now also U$2.P$6; no longer SV2.6
- net N$21: no longer C10.1
- net N$24: now also U$3.1; no longer POWERIN.P
- net SCK: now also U$2.P$5; no longer SV2.5

Commit message: Revert "V0.9 Layout and Schematic ready for review and version jump to 1.0."
This reverts commit 28fefd69818988460ab9c4da467096be04e20f85.
Parts:
- removed U$2: HEADER1,27, SkateMateMagicGlove:HEADER1,27
- removed U$3: MICRO-USB-ZX62R-B-5P, con-hirose:MICRO-USB-ZX62R-B-5P
- added C10: 4.7u, eagle-ltspice:CC0603
- added C4, C5: 22p, eagle-ltspice:CC0603
- added POWERIN: +, wirepad:1,6/0,8
- added SV2: RFM75, con-lstb:MA08-1
- added Y1: 8MHz, crystals:ABM3
Connections:
- new net N$3: C5.2, U1.PB7, Y1.1
- new net N$4: C4.2, U1.PB6, Y1.2
- net +3V3: now also SV2.2; no longer U$2.P$2
- net CE: now also SV2.3; no longer U$2.P$3
- net CSN: now also SV2.4; no longer U$2.P$4
- net GND: now also C10.2, C4.1, C5.1, SV2.1; no longer U$2.P$1
- net IRQ: now also SV2.8; no longer U$2.P$8
- net MISO: now also SV2.7; no longer U$2.P$7
- net MOSI: now also SV2.6; no longer U$2.P$6
- net N$21: now also C10.1
- net N$24: now also POWERIN.P; no longer U$3.1
- net SCK: now also SV2.5; no longer U$2.P$5
