File: src/skatemate_proto.brd (EAGLE design)
At the start: 160 x 100 mm, 89 parts, among them IC1 REG1117, Q1 IRF740, Q2 IRF740, Q3 IRF740, Q4 IRF740, Q5 IRF740, Q6 IRF740, U1 DRV8301DCAR

Commit message: more layout
Parts:
- moved J1 85.4 mm to (4.06, 5.84), turned to 270 degrees
- moved R23 81.1 mm to (10.9, 1.52), turned to 180 degrees
- moved R24 71.9 mm to (10.9, 6.60)
- moved R25 65.8 mm to (10.9, 8.64)
- moved R26 65.8 mm to (10.9, 4.57)
- moved R27 55.7 mm to (10.9, 10.7)
- moved C16 1.44 mm to (58.9, 38.1), turned to 90 degrees
Routing:
- net N$22: track 0.00 -> 10.6 mm
- net N$25: track 0.00 -> 8.56 mm
- net GND: track 150.0 -> 158.4 mm, vias 27 -> 28
- net N$24: track 0.00 -> 7.09 mm
- net N$23: track 0.00 -> 6.22 mm
- net VCC: track 170.4 -> 172.0 mm, vias 9 -> 10
- net N$18: track 6.50 -> 7.38 mm

Commit message: Verdrohtet
Parts:
- moved C29 3.98 mm to (23.9, 17.8)
- moved C31 3.98 mm to (21.8, 17.8)
- moved C32 0.25 mm to (6.35, 23.4)
Routing:
- net VCC: track 172.0 -> 308.1 mm, vias 10 -> 15
- net GND: track 158.4 -> 246.5 mm, vias 28 -> 34
- net USB_D+: track 13.3 -> 41.7 mm, vias 1 -> 4
- net USB_D-: track 10.9 -> 36.1 mm, vias 1 -> 4
- net SWDIO: track 20.1 -> 23.5 mm
- net N$23: track 6.22 -> 8.26 mm
- net SSENSE: track 113.5 -> 115.1 mm
- net CSENSE: track 122.0 -> 122.8 mm
- net ASENSE: track 156.5 -> 157.2 mm
- net BSENSE: track 138.9 -> 139.6 mm
