File: MotorControl/skatemate_proto.brd (EAGLE design)
At the start: 126.5 x 87.3 mm, 104 parts, among them IC1 REG1117, Q1 IRF740, Q2 IRF740, Q3 IRF740, Q4 IRF740, Q5 IRF740, Q6 IRF740, U1 DRV8301DCAR

Commit message: added USART TX/RX labels
Connections:
- new net USART3_RX: U$3.30
- new net USART3_TX: U$3.29
Changed lines of the file:
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@@
 <wire x1="6.98" y1="30.358" x2="8.664" y2="28.674" width="0.254" layer="1"/>
+</signal>
+<signal name="USART3_RX">
+<contactref element="U$3" pad="30"/>
+</signal>
+<signal name="USART3_TX">
+<contactref element="U$3" pad="29"/>
 </signal>
 </signals>
