File: MagicGlove/Extern Print/SkateMate_Glove_Extern.sch (EAGLE design)
At the start: 42 parts, among them IC1 BU33TD3WG, IC2 LMV321M5, U2 ATMEGA328PB-AU

Commit message: Backup commit.
Connections:
- net +3V3: now also SV1.2; no longer SV1.5
- net GND: now also SV1.6; no longer SV1.1
- net MISO: now also SV1.1; no longer SV1.6
- net MOSI: now also SV1.4; no longer SV1.3
- net RESETICSP: now also SV1.5; no longer SV1.2
- net SCK: now also SV1.3; no longer SV1.4
Other:
- moved on the sheet: SV1
Changed lines of the file:
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@@
 <instance part="R5" gate="G$1" x="101.6" y="45.72" rot="R180"/>
 <instance part="GND6" gate="1" x="20.32" y="71.12" rot="R180"/>
-<instance part="SV1" gate="1" x="182.88" y="30.48"/>
+<instance part="SV1" gate="1" x="182.88" y="30.48" rot="R180"/>
 <instance part="GND1" gate="1" x="193.04" y="25.4"/>
 <instance part="+3V31" gate="G$1" x="195.58" y="33.02" rot="R270"/>
@@
 </segment>
 <segment>
-<pinref part="SV1" gate="1" pin="1"/>
+<pinref part="SV1" gate="1" pin="6"/>
 <wire x1="190.5" y1="27.94" x2="193.04" y2="27.94" width="0.1524" layer="91"/>
 <pinref part="GND1" gate="1" pin="GND"/>
@@
 </segment>
 <segment>
-<pinref part="SV1" gate="1" pin="5"/>
+<pinref part="SV1" gate="1" pin="2"/>
 <pinref part="+3V31" gate="G$1" pin="+3V3"/>
 <wire x1="193.04" y1="33.02" x2="190.5" y2="33.02" width="0.1524" layer="91"/>
@@
 </segment>
 <segment>
-<pinref part="SV1" gate="1" pin="2"/>
+<pinref part="SV1" gate="1" pin="5"/>
 <wire x1="175.26" y1="27.94" x2="166.37" y2="27.94" width="0.1524" layer="91"/>
 <label x="166.37" y="27.94" size="0.6096" layer="95" rot="R180" xref="yes"/>
@@
 </segment>
 <segment>
-<pinref part="SV1" gate="1" pin="4"/>
+<pinref part="SV1" gate="1" pin="3"/>
 <wire x1="175.26" y1="30.48" x2="166.37" y2="30.48" width="0.1524" layer="91"/>
 <label x="166.37" y="30.48" size="0.6096" layer="95" rot="R180" xref="yes"/>
@@
 </segment>
 <segment>
-<pinref part="SV1" gate="1" pin="6"/>
+<pinref part="SV1" gate="1" pin="1"/>
 <wire x1="175.26" y1="33.02" x2="166.37" y2="33.02" width="0.1524" layer="91"/>
 <label x="166.37" y="33.02" size="0.6096" layer="95" rot="R180" xref="yes"/>
@@
 </segment>
 <segment>
-<pinref part="SV1" gate="1" pin="3"/>
+<pinref part="SV1" gate="1" pin="4"/>
 <wire x1="190.5" y1="30.48" x2="195.58" y2="30.48" width="0.1524" layer="91"/>
 <label x="195.58" y="30.48" size="0.6096" layer="95" xref="yes"/>
