File: BatteryManagment/BM_ pre.brd (EAGLE design)
At the start: 107.7 x 100 mm, 123 parts, among them IC1 LMV321M5, U1 ATMEGA328P-AU, U2 LTC4440EMS8E-5PBF

Commit message: schematic up to date
Parts:
- added R57: 10k, rcl:R0603
Connections:
- new net N$45: R57.2, U$26.1
- net UC_M_CONT: now also R57.1; no longer U$26.1
Routing:
- net UC_M_CONT: track 79.8 -> 61.7 mm, vias 2 -> 1
- net N$45: track 0.00 -> 17.3 mm, vias 0 -> 1
Changed lines of the file:
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@@
 <element name="U$20" library="BM_pre" package="Z03A" value="BC327" x="91.85" y="92.44" rot="R90"/>
 <element name="U$21" library="BM_pre" package="Z03A" value="BC327" x="91.86" y="97.24" rot="R90"/>
+<element name="R57" library="rcl" package="R0603" value="10k" x="49.95" y="48.06" rot="MR180"/>
 </elements>
 <signals>
@@
 <signal name="CHARGE_CONTROL">
 <contactref element="U$2" pad="1"/>
-<wire x1="22.25" y1="30.31" x2="19.66" y2="27.72" width="0.45" layer="1"/>
+<wire x1="22.55" y1="30.61" x2="19.66" y2="27.72" width="0.45" layer="1"/>
 <wire x1="19.66" y1="27.72" x2="18.5725" y2="27.72" width="0.3" layer="1"/>
 <wire x1="18.5725" y1="27.72" x2="18.4925" y2="27.64" width="0.3" layer="1"/>
-<wire x1="22.55" y1="30.61" x2="22.25" y2="30.31" width="0.45" layer="1"/>
 <contactref element="U2" pad="7"/>
 <contactref element="C12" pad="2"/>
-<wire x1="22.765" y1="33.8102" x2="22.78" y2="33.8102" width="0.3" layer="1"/>
-<wire x1="22.78" y1="32.63" x2="22.55" y2="32.4" width="0.45" layer="1"/>
+<wire x1="22.78" y1="33.8102" x2="22.765" y2="33.8102" width="0.3" layer="1"/>
 <wire x1="22.55" y1="32.4" x2="22.55" y2="31.7" width="0.45" layer="1"/>
-<wire x1="22.78" y1="33.8102" x2="22.78" y2="32.63" width="0.45" layer="1"/>
 <wire x1="22.55" y1="31.7" x2="22.55" y2="30.61" width="0.45" layer="1"/>
+<wire x1="22.765" y1="33.8102" x2="22.765" y2="32.615" width="0.45" layer="1"/>
+<wire x1="22.765" y1="32.615" x2="22.55" y2="32.4" width="0.45" layer="1"/>
 </signal>
 <signal name="MOTOR_CONTROL">
@@
 <wire x1="45.8414" y1="82.31" x2="45.8652" y2="82.3338" width="0.3" layer="1"/>
 <wire x1="35.14" y1="48.645" x2="35.14" y2="84.29" width="0.3" layer="1"/>
-<contactref element="U$26" pad="1"/>
-<via x="62.84" y="42.58" extent="1-16" drill="0.5"/>
-<wire x1="62.84" y1="42.58" x2="62.84" y2="40.51" width="0.3" layer="1"/>
-<wire x1="62.84" y1="40.51" x2="62.85" y2="40.5" width="0.3" layer="1"/>
-<wire x1="35.715" y1="48.07" x2="57.35" y2="48.07" width="0.3" layer="16"/>
-<wire x1="57.35" y1="48.07" x2="62.84" y2="42.58" width="0.3" layer="16"/>
+<contactref element="R57" pad="1"/>
+<wire x1="35.715" y1="48.07" x2="49.09" y2="48.07" width="0.3" layer="16"/>
+<wire x1="49.09" y1="48.07" x2="49.1" y2="48.06" width="0.3" layer="16" curve="-90"/>
 </signal>
 <signal name="CHARGE_PWM">
@@
 <wire x1="74.07" y1="74.36" x2="73.88" y2="74.17" width="0.3" layer="16"/>
 </signal>
+<signal name="N$45">
+<contactref element="U$26" pad="1"/>
+<contactref element="R57" pad="2"/>
+<wire x1="50.8" y1="48.06" x2="58.9" y2="48.06" width="0.3" layer="16"/>
+<wire x1="58.9" y1="48.06" x2="62.84" y2="44.12" width="0.3" layer="16"/>
+<wire x1="62.84" y1="44.12" x2="62.84" y2="43.65" width="0.3" layer="16"/>
+<via x="62.84" y="43.65" extent="1-16" drill="0.6"/>
+<wire x1="62.84" y1="43.65" x2="62.84" y2="40.51" width="0.3" layer="1"/>
+<wire x1="62.84" y1="40.51" x2="62.85" y2="40.5" width="0.3" layer="1"/>
+</signal>
 </signals>
