File: BatteryManagment/BM_v2.brd (EAGLE design)
At the start: 81 x 60 mm, 163 parts, among them U1 ATMEGA328P-AU

Commit message: little update
Parts:
- moved C15 0.35 mm to (7.18, 37.3)
- flipped CELL1 to the bottom
- flipped CELL2 to the bottom
- flipped CELL3 to the bottom
- flipped CELL4 to the bottom
- flipped CELL5 to the bottom
- flipped CELL6 to the bottom
Changed lines of the file:
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@@
 </element>
 <element name="C14" library="rcl" package="C0603" value="100nF" x="6.92" y="13.9" rot="MR180"/>
-<element name="C15" library="rcl" package="E3,5-10" value="100u" x="7.27" y="37.67" rot="MR90"/>
+<element name="C15" library="rcl" package="E3,5-10" value="100u" x="7.18" y="37.33" rot="MR90"/>
 <element name="C16" library="rcl" package="C0603" value="100nF" x="6.68" y="16.54" rot="MR270"/>
 <element name="C2" library="rcl" package="C0603" value="100n" x="24.1" y="11.66" rot="R270"/>
@@
 <element name="C7" library="rcl" package="C0603" value="100n" x="66.64" y="9.55"/>
 <element name="C9" library="rcl" package="C0805" value="10u" x="-40.64" y="85.09"/>
-<element name="CELL1" library="wirepad" package="SMD2,54-5,08" value="" x="62.24" y="56.91" rot="R180"/>
-<element name="CELL2" library="wirepad" package="SMD2,54-5,08" value="" x="58.77" y="56.94" rot="R180"/>
-<element name="CELL3" library="wirepad" package="SMD2,54-5,08" value="" x="55.27" y="56.94" rot="R180"/>
-<element name="CELL4" library="wirepad" package="SMD2,54-5,08" value="" x="51.69" y="56.95" rot="R180"/>
-<element name="CELL5" library="wirepad" package="SMD2,54-5,08" value="" x="48.32" y="56.93" rot="R180"/>
-<element name="CELL6" library="wirepad" package="SMD2,54-5,08" value="" x="44.87" y="56.93" rot="R180"/>
+<element name="CELL1" library="wirepad" package="SMD2,54-5,08" value="" x="62.24" y="56.91" rot="MR180"/>
+<element name="CELL2" library="wirepad" package="SMD2,54-5,08" value="" x="58.77" y="56.94" rot="MR180"/>
+<element name="CELL3" library="wirepad" package="SMD2,54-5,08" value="" x="55.27" y="56.94" rot="MR180"/>
+<element name="CELL4" library="wirepad" package="SMD2,54-5,08" value="" x="51.69" y="56.95" rot="MR180"/>
+<element name="CELL5" library="wirepad" package="SMD2,54-5,08" value="" x="48.32" y="56.93" rot="MR180"/>
+<element name="CELL6" library="wirepad" package="SMD2,54-5,08" value="" x="44.87" y="56.93" rot="MR180"/>
 <element name="EXT_LED1" library="wirepad" package="SMD2,54-5,08" value="" x="7.2" y="56.89"/>
 <element name="EXT_LED2" library="wirepad" package="SMD2,54-5,08" value="" x="10.82" y="56.84"/>
@@
 <wire x1="24.1" y1="10.81" x2="13.98" y2="16.8039" width="0" layer="19" extent="1-16"/>
 <wire x1="30.22" y1="6.712" x2="24.1" y2="10.81" width="0" layer="19" extent="1-1"/>
-<wire x1="7.27" y1="39.448" x2="21.135" y2="33.73" width="0" layer="19" extent="1-1"/>
+<wire x1="7.18" y1="39.108" x2="21.135" y2="33.73" width="0" layer="19" extent="1-1"/>
 <wire x1="67.49" y1="9.55" x2="56.705" y2="34.26" width="0" layer="19" extent="1-1"/>
 <wire x1="74.34" y1="4.71" x2="67.49" y2="9.55" width="0" layer="19" extent="1-1"/>
 <wire x1="61.42" y1="3.662" x2="67.49" y2="9.55" width="0" layer="19" extent="1-1"/>
-<wire x1="-18.1" y1="68.75" x2="7.27" y2="39.448" width="0" layer="19" extent="1-1"/>
+<wire x1="-18.1" y1="68.75" x2="7.18" y2="39.108" width="0" layer="19" extent="1-1"/>
 <wire x1="-15.56" y1="76.37" x2="-18.1" y2="68.75" width="0" layer="19" extent="1-1"/>
 <wire x1="-21.91" y1="76.37" x2="-15.56" y2="76.37" width="0" layer="19" extent="1-1"/>
@@
 <contactref element="U$35" pad="P$2"/>
 <contactref element="15V" pad="1"/>
-<wire x1="7.27" y1="35.892" x2="3.66" y2="56.85" width="0" layer="19" extent="1-1"/>
-<wire x1="7.3" y1="28.77" x2="7.27" y2="35.892" width="0" layer="19" extent="16-16"/>
+<wire x1="7.18" y1="35.552" x2="3.66" y2="56.85" width="0" layer="19" extent="1-1"/>
+<wire x1="7.3" y1="28.77" x2="7.18" y2="35.552" width="0" layer="19" extent="16-16"/>
 <wire x1="6.68" y1="17.39" x2="7.3" y2="28.77" width="0" layer="19" extent="16-16"/>
 <wire x1="4.5" y1="17.39" x2="6.68" y2="17.39" width="0" layer="19" extent="16-16"/>

Commit message: next generation
Parts:
- moved U$15 181.7 mm to (67.3, 52.3), flipped to the bottom
- moved U$16 176.6 mm to (62.3, 52.3), flipped to the bottom
- moved U$17 171.8 mm to (57.3, 52.3), flipped to the bottom
- moved U$18 167.4 mm to (52.3, 52.3), flipped to the bottom
- moved R82 163.4 mm to (52.3, 57.8), turned to 270 degrees
- moved U$20 163.3 mm to (47.3, 52.3), flipped to the bottom
- moved R79 163.2 mm to (67.3, 57.8), turned to 270 degrees
- moved R81 161.4 mm to (55.2, 57.8), turned to 90 degrees
- moved U$21 159.5 mm to (42.3, 52.3), flipped to the bottom
- moved U$29 158.7 mm to (53.8, 44.8), flipped to the bottom, turned to 90 degrees
- moved R80 158.6 mm to (57.3, 57.8), turned to 270 degrees
- moved R43 157.6 mm to (47.4, 49.2), flipped to the bottom
- moved R42 157.5 mm to (52.4, 49.2), flipped to the bottom
- moved R41 157.4 mm to (57.4, 49.2), flipped to the bottom
- moved R40 157.3 mm to (62.4, 49.2), flipped to the bottom
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
Commit message: update save
Parts:
- removed GND14: (no value), wirepad:SMD2,54-5,08
- added U$23: EATON_50A_FUSE, BM_pre:LITTELFUSE
- moved R57 15.8 mm to (20.1, 18.8)
- moved C16 14.8 mm to (15.2, 28.7), turned to 180 degrees
- moved U1 1.85 mm to (31.5, 46.5), turned to 270 degrees
- turned R81 to 270 degrees
Connections:
- removed net +12V: R88.2, U$37.1
- new net N$73: BATTERY+.P$1, U$23.P$3
- net +15V: now also R88.2, U$37.1
- net BATTERY+: now also C14.2, U$1.2, U$23.P$1; no longer BATTERY+.P$1
- net GND: no longer GND14.1
- net VCC: no longer C14.2, U$1.2
Routing:
- net +15V: track 0.00 -> 29.2 mm
- net N$21: track 0.00 -> 18.3 mm
- net CELL2: track 0.00 -> 17.2 mm, vias 0 -> 2
- net CELL1: track 0.00 -> 16.9 mm, vias 0 -> 2
- net CELL3: track 0.00 -> 16.9 mm, vias 0 -> 2
- net VCC: track 0.00 -> 16.9 mm
- net CELL4: track 0.00 -> 16.8 mm, vias 0 -> 2
- net CELL5: track 0.00 -> 16.2 mm, vias 0 -> 2
- net N$45: track 0.00 -> 12.1 mm
- net CURRENT-: track 0.00 -> 11.6 mm
- net CELL6: track 0.00 -> 8.88 mm, vias 0 -> 1
- net BATTERY+: track 0.00 -> 5.79 mm
- net N$14: track 0.00 -> 4.98 mm, vias 0 -> 1
- net FEEDBACK: track 0.00 -> 4.93 mm
- net N$5: track 0.00 -> 4.75 mm, vias 0 -> 1
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- added copper zone on layer 1, net BATTERY+
- added copper zone on layer 1, net CURRENT+
- added copper zone on layer 1, net CURRENT-
- added copper zone on layer 1, net N$73
- added copper zone on layer 1, net TS
- added copper zone on layer 1, net VCC

Commit message: backup
Parts:
- removed R73: (no value), rcl:R0603
- moved R39 116.3 mm to (62.3, 33.4), flipped to the bottom, turned to 180 degrees
- moved R75 101.7 mm to (52.5, -1.77)
- moved R1 97.3 mm to (69.7, 26.8), turned to 270 degrees
- moved U$26 91.9 mm to (58.7, 32.2), flipped to the bottom, turned to 180 degrees
- moved R37 79.4 mm to (30.7, 40.6), turned to 180 degrees
- moved R36 75.4 mm to (30.2, 38.1), turned to 270 degrees
- moved R20 73.4 mm to (33.0, 55.4), turned to 180 degrees
- moved C13 46.4 mm to (28.1, 40.1), turned to 90 degrees
- moved R74 38.8 mm to (18.9, 49.2), turned to 90 degrees
- moved U1 3.27 mm to (28.5, 47.8)
- moved C11 2.27 mm to (45.5, 37.3), turned to 0 degrees
- moved U$19 2.18 mm to (45.5, 32.2), turned to 0 degrees
- moved U$8 1.99 mm to (40.9, 35.7)
- moved PAD2 1.73 mm to (49.9, 31.7), turned to 90 degrees
- moved R29 1.17 mm to (40.7, 30.4)
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Connections:
- removed net N$57: R73.2, U$36.4
- net EN_LED: now also U$36.4; no longer R73.1
Routing:
- net +5V: track 0.00 -> 53.9 mm, vias 0 -> 2
- net V_MEAS: track 0.00 -> 52.3 mm, vias 0 -> 2
- net ADC_BAT_1: track 0.00 -> 50.2 mm, vias 0 -> 2
- net C1_B: track 0.00 -> 46.3 mm, vias 0 -> 1
- net UC_M_CONT: track 0.00 -> 46.2 mm, vias 0 -> 1
- net C2_B: track 0.00 -> 41.5 mm, vias 0 -> 1
- net ADC_BAT_2: track 0.00 -> 39.7 mm, vias 0 -> 2
- net C3_B: track 0.00 -> 36.4 mm, vias 0 -> 1
- net C6_B: track 0.00 -> 35.8 mm, vias 0 -> 1
- net C4_B: track 0.00 -> 35.3 mm, vias 0 -> 1
- net ADC_BAT_3: track 0.00 -> 33.7 mm, vias 0 -> 2
- net CURRENTSENSE: track 0.00 -> 33.3 mm, vias 0 -> 2
- net C5_B: track 0.00 -> 31.7 mm, vias 0 -> 1
- net ADC_BAT_4: track 0.00 -> 28.5 mm, vias 0 -> 2
- net RESETICSP: track 0.00 -> 27.0 mm
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- added copper zone on layer 1, net MOTOR+
Other:
- board size 81 x 60 mm -> 81 x 61 mm

Commit message: finish layout
Parts:
- moved R75 55.6 mm to (13.5, 37.8), turned to 90 degrees
- moved R9 1.08 mm to (46.4, 51.1), turned to 180 degrees
- moved R6 1.04 mm to (56.4, 51.1), turned to 180 degrees
- moved R8 1.02 mm to (51.4, 51.1), turned to 180 degrees
- moved R4 0.87 mm to (61.4, 51.8), turned to 180 degrees
- moved R38 0.86 mm to (66.4, 51.9), turned to 180 degrees
- moved C13 0.24 mm to (27.9, 40.1)
Routing:
- net GND: track 12.6 -> 141.1 mm, vias 0 -> 44
- net BATTERY+: track 11.7 -> 87.3 mm, vias 0 -> 4
- net EN_15V: track 0.00 -> 40.3 mm, vias 0 -> 1
- net SELBSTERHALTUNG: track 5.38 -> 33.5 mm, vias 1 -> 2
- net +15V: track 46.3 -> 69.1 mm
- net VCC: track 16.9 -> 38.5 mm, vias 0 -> 2
- net +5V: track 53.9 -> 73.9 mm, vias 2 -> 3
- net MOSI: track 18.0 -> 34.5 mm, vias 1 -> 2
- net SCK: track 4.50 -> 19.8 mm, vias 0 -> 2
- net TS: track 1.70 -> 9.02 mm
- net N$37: track 0.07 -> 3.16 mm
- net MISO: track 26.0 -> 29.0 mm
- net CELL4: track 15.6 -> 18.6 mm, vias 1 -> 2
- net CELL3: track 16.3 -> 19.2 mm, vias 1 -> 2
- net N$33: track 0.00 -> 2.73 mm
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- added copper zone on layer 1, net GND
- added copper zone on layer 16, net GND
Other:
- board size 81 x 61 mm -> 81 x 61.5 mm
