File: BatteryManagment/BM_v2.sch (EAGLE design)
At the start: 123 parts, among them IC1 LMV321M5, U1 ATMEGA328P-AU, U2 LTC4440EMS8E-5PBF

Commit message: Update
Parts:
- added C1: 10nF, rcl:C-EUC0603
- added C14: 100nF, rcl:C-EUC0603
- added C17: 100u, rcl:CPOL-EUE3.5-10
- added R59, R60: (no value), rcl:R-EU_R0603
- added U$1: LM22677TJE-ADJ/NOPB, BM_pre:LM22677TJE-ADJ/NOPB
- added U$33: BAS16, BM_pre:BAS16
Connections:
- new net +15V: R59.2
- new net FEEDBACK: R59.1, R60.2, U$1.FB
- new net N$1: C1.2, U$1.BOOT
- new net VCC: C14.2, C17.+, C2.1, C3.1, C4.+, R36.2, U$1.VIN, U$2.S, U$32.C, VIN.TP
- net GND: now also C14.1, C17.-, R60.1, U$1.GND, U$10.E, U$11.E, U$12.E, U$13.E, U$14.E, U$33.A, U$9.E
- net N$21: now also C1.1, U$1.SW, U$33.C; no longer U$10.E, U$11.E, U$12.E, U$13.E, U$14.E, U$9.E
- net VIN_SENSE: no longer C2.1, C3.1, C4.+, R36.2, U$2.S, U$32.C, VIN.TP

Commit message: schematic up to date
Parts:
- removed IC1: LMV321M5, BM_pre:LMV321M5
- removed L1: 2310-V-RC, BM_pre:2310-V-RC
- removed U2: LTC4440EMS8E-5PBF, BM_pre:LTC4440EMS8E-5PBF
- added 15V, EXT_LED1, EXT_LED2, EXT_LED3: (no value), wirepad:SMD5
- added C15: 100u, rcl:CPOL-EUE3.5-10
- added C16: 100nF, rcl:C-EUC0603
- added R57, R58, R61, R62, R63, R64, R65, R66, R67, R68, R69, R70, R71, R72, R73, R76, R77, R78, R79, R80, R81, R82, R83, R84, R85, R86, R87: (no value), rcl:R-EU_R0603
- added R74, R75: 0, rcl:R-EU_R0603
- added U$34: COIL_PVC-2, BM_pre:COIL_PVC-2
- added U$35: SRN1060, BM_pre:SRN1060
- added U$36: SI4490, BM_pre:SI4490
- added U$37: FAN73711, BM_pre:FAN73711
- added U$38: LM2904, BM_pre:LM2904
- U$19: value IRF9310PBF -> FDN340; device BM_pre:IRF9310PBF -> BM_pre:FDN340
Connections:
- new net EN_15V: R75.1, U$1.EN
- new net EN_LED: R73.1, R74.1
- new net N$45: R57.2, U$1.DAP
- new net N$46: R58.2, U$1.RT/SYNC
- new net N$47: EXT_LED1.P, R61.2, R63.2
- new net N$48: R61.1, R62.2
- new net N$49: R63.1, R64.2
- new net N$50: EXT_LED2.P, R65.2, R66.2
- new net N$51: R65.1, R67.2
- new net N$52: R66.1, R68.2
- new net N$53: R62.1, R64.1, R67.1, R68.1, R71.1, R72.1, U$36.D
- new net N$54: EXT_LED3.P, R69.2, R70.2
- new net N$55: R69.1, R71.2
- new net N$56: R70.1, R72.2
- new net N$57: R73.2, U$36.G
- new net N$58: R15.1, R77.2
- new net N$59: R31.1, R76.2
- new net N$60: R2.1, R78.2
- new net N$61: R14.1, R79.2
- new net N$62: R16.2, R80.2
- new net N$63: R32.2, R81.2
- new net N$64: R17.2, R82.2
- new net N$65: R33.2, R83.2
- new net N$66: R18.2, R84.2
- new net N$67: R34.2, R85.2
- new net N$68: R19.2, R86.2
- new net N$69: R35.2, R87.2
- net +12V: now also U$37.VDD; no longer U2.VCC
- net +15V: now also 15V.P, C15.+, C16.1, R57.1, U$35.2
- net +5V: now also U$38A.V+; no longer IC1.V+
- net CELL1: now also R76.1, R77.1; no longer R15.1, R31.1
- net CELL2: now also R80.1, R81.1; no longer R16.2, R32.2
- net CELL3: now also R82.1, R83.1; no longer R17.2, R33.2
- net CELL4: now also R84.1, R85.1; no longer R18.2, R34.2
- net CELL5: now also R86.1, R87.1; no longer R19.2, R35.2
- net CHARGE_CONTROL: now also U$37.HOUT; no longer U2.TG
- net CHARGE_PWM: now also U$37.IN, U1.PD6; no longer U1.PB6, U2.INP
- net CURRENT+: now also U$34.1; no longer L1.2
- net CURRENTSENSE: now also U$38A.OUT; no longer IC1.OUT
- net GND: now also C15.-, C16.2, R58.1, R78.1, R79.1, U$36.S, U$37.GND, U$37.NC, U$37.NC_, U$38A.V-, U$38B.+IN, U$38B.-IN; no longer IC1.V-, R14.1, R2.1, U2.GND, U2.GND_2, U2.NC
- net MISO: now also R74.2
- net MOSI: now also R75.2
- net N$15: now also U$38A.+IN; no longer IC1.+IN
- net N$16: now also U$38A.-IN; no longer IC1.-IN
- net N$2: now also U$37.VS; no longer U2.BOOST
- net N$21: now also U$35.1
- net TS: now also U$34.2, U$37.VB; no longer L1.1, U2.TS
- net V_MEAS: now also U1.PB6; no longer U1.PD6
Other:
- moved on the sheet: C1, C14, C17, R21, R22, R23, R24, R59, R60, U$1, U$33

Commit message: Start with schematic
Parts:
- removed C10: 10u, rcl:C-EUC0805
- removed C17: 100u, rcl:CPOL-EUE3.5-10
- removed C6: 47u, rcl:C-EUC1812
- removed C8: 1u_100V, rcl:C-EUC1206
- removed D1: 1N4004, diode:1N4004
- removed U$23: IPB180P04P4L-02, BM_pre:IPB180P04P4L-02
- added R88: 39k, rcl:R-EU_R0603
- added R89: (no value), rcl:R-EU_R0603
- C3: value 47u -> 100n; device rcl:C-EUC1812 -> rcl:C-EUC0603
- U$15, U$16, U$17, U$18, U$20, U$21: value BC327 -> FDN340; device BM_pre:BC327 -> BM_pre:FDN340
- U$7: value ZXTR2012Z -> BAV99; device BM_pre:ZXTR2012Z -> BM_pre:BAV99
Connections:
- removed net VIN_SENSE: C8.1, U$7.VI
- new net N$70: R88.1, U$7.A
- new net N$71: R89.2, U$37.HOUT
- net +12V: now also R88.2; no longer C10.1, D1.A, U$7.VO
- net BATTERY+: no longer U$23.S
- net CELL1: now also U$15.S; no longer U$15.E
- net CELL2: now also U$16.S; no longer U$16.E
- net CELL3: now also U$17.S; no longer U$17.E
- net CELL4: now also U$18.S; no longer U$18.E
- net CELL5: now also U$20.S; no longer U$20.E
- net CELL6: now also U$21.S; no longer U$21.E
- net CHARGE_CONTROL: now also R89.1; no longer C12.2, U$37.HOUT
- net CURRENT-: no longer C6.1
- net CURRENTSENSE: now also C3.1
- net GND: no longer C10.2, C17.-, C6.2, C8.2, U$7.GND
- net MOTOR+: no longer U$23.D
- net MOTOR_CONTROL: no longer U$23.G
- net N$11: now also U$17.D; no longer U$17.C
- net N$12: now also U$18.D; no longer U$18.C
- net N$13: now also U$20.D; no longer U$20.C
- net N$14: now also U$21.D; no longer U$21.C
- net N$2: now also U$7.C; no longer D1.C
- net N$22: now also U$15.G; no longer U$15.B
- net N$28: now also U$16.G; no longer U$16.B
- net N$29: now also U$17.G; no longer U$17.B
- net N$30: now also U$18.G; no longer U$18.B
- net N$31: now also U$20.G; no longer U$20.B
- net N$32: now also U$21.G; no longer U$21.B
- net N$5: now also U$15.D; no longer U$15.C
- net N$6: now also U$16.D; no longer U$16.C
- net TS: now also C12.2, U$2.S; no longer U$2.D
- net VCC: now also U$2.D; no longer C17.+, C3.1, U$2.S

Commit message: next generation
Changed lines of the file:
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@@
 <wire x1="160.02" y1="55.88" x2="149.86" y2="55.88" width="0.1524" layer="91"/>
 <pinref part="U$19" gate="G$1" pin="G"/>
+<junction x="149.86" y="55.88"/>
 </segment>
 </net>

Commit message: update save
Parts:
- removed GND14: (no value), wirepad:SMD5
- added U$23: EATON_50A_FUSE, BM_pre:EATON_50A_FUSE
Connections:
- removed net +12V: R88.2, U$37.VDD
- new net N$73: BATTERY+.TP, U$23.2A
- net +15V: now also R88.2, U$37.VDD
- net BATTERY+: now also C14.2, U$1.VIN, U$23.1A; no longer BATTERY+.TP
- net GND: no longer GND14.P
- net VCC: no longer C14.2, U$1.VIN
Changed lines of the file:
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@@
 <part name="R24" library="rcl" deviceset="R-EU_" device="R0603" value="66k"/>
 <part name="C12" library="rcl" deviceset="C-EU" device="C0603" value="100n"/>
-<part name="P+7" library="supply1" deviceset="+12V" device=""/>
 <part name="GND19" library="supply1" deviceset="GND" device=""/>
 <part name="LED2" library="eagle-ltspice" deviceset="LED_E" device=""/>
@@
 <part name="GND22" library="supply1" deviceset="GND" device=""/>
 <part name="CELL1" library="wirepad" deviceset="SMD5" device=""/>
-<part name="GND14" library="wirepad" deviceset="SMD5" device=""/>
 <part name="CELL2" library="wirepad" deviceset="SMD5" device=""/>
 <part name="CELL3" library="wirepad" deviceset="SMD5" device=""/>
@@
 <part name="P+9" library="supply1" deviceset="VCC" device=""/>
 <part name="P+10" library="supply1" deviceset="VCC" device=""/>
-<part name="P+11" library="supply1" deviceset="VCC" device=""/>
 <part name="C1" library="rcl" deviceset="C-EU" device="C0603" value="10nF"/>
 <part name="C14" library="rcl" deviceset="C-EU" device="C0603" value="100nF"/>
@@
 <part name="R89" library="rcl" deviceset="R-EU_" device="R0603"/>
 <part name="GND8" library="supply1" deviceset="GND" device=""/>
+<part name="U$23" library="BM_pre" deviceset="EATON_50A_FUSE" device=""/>
+<part name="P+2" library="supply1" deviceset="+15V" device=""/>
 </parts>
 <sheets>
@@
 <instance part="U$34" gate="G$1" x="116.84" y="129.54"/>
 <instance part="U$19" gate="G$1" x="152.4" y="68.58" rot="MR90"/>
+<instance part="U$23" gate="G$1" x="172.72" y="152.4" rot="R90"/>
 </instances>
 <busses>
@@
 <wire x1="185.42" y1="121.92" x2="185.42" y2="129.54" width="0.1524" layer="91"/>
 <junction x="185.42" y="129.54"/>
-<pinref part="BATTERY+" gate="G$1" pin="TP"/>
-<wire x1="172.72" y1="162.56" x2="172.72" y2="129.54" width="0.1524" layer="91"/>
-<label x="172.72" y="157.48" size="1.778" layer="95" rot="R180" xref="yes"/>
+<label x="172.72" y="137.16" size="1.778" layer="95" rot="R180" xref="yes"/>
 <junction x="172.72" y="129.54"/>
+<pinref part="U$23" gate="G$1" pin="1A"/>
+<wire x1="172.72" y1="147.32" x2="172.72" y2="129.54" width="0.1524" layer="91"/>
 </segment>
 <segment>
@@
 </segment>
 </net>
+<net name="N$73" class="0">
+<segment>
+<pinref part="BATTERY+" gate="G$1" pin="TP"/>
+<wire x1="172.72" y1="162.56" x2="172.72" y2="157.48" width="0.1524" layer="91"/>
+<pinref part="U$23" gate="G$1" pin="2A"/>
+</segment>
+</net>
 </nets>
 </sheet>
@@
 <instances>
 <instance part="FRAME1" gate="G$1" x="0" y="0"/>
-<instance part="GND15" gate="1" x="139.7" y="132.08"/>
+<instance part="GND15" gate="1" x="149.86" y="132.08"/>
 <instance part="R3" gate="G$1" x="116.84" y="157.48" rot="R90"/>
 <instance part="R4" gate="G$1" x="109.22" y="180.34" rot="R90"/>
@@
 <instance part="R24" gate="G$1" x="76.2" y="55.88" rot="R180"/>
 <instance part="C12" gate="G$1" x="294.64" y="58.42" rot="R90"/>
-<instance part="P+7" gate="1" x="223.52" y="93.98"/>
 <instance part="GND19" gate="1" x="226.06" y="12.7"/>
 <instance part="CELL1" gate="1" x="139.7" y="180.34" rot="R270"/>
-<instance part="GND14" gate="1" x="139.7" y="172.72" rot="R270"/>
 <instance part="CELL2" gate="1" x="139.7" y="187.96" rot="R270"/>
 <instance part="CELL3" gate="1" x="139.7" y="195.58" rot="R270"/>
@@
 <instance part="R89" gate="G$1" x="317.5" y="60.96" rot="R180"/>
 <instance part="GND8" gate="1" x="119.38" y="45.72"/>
+<instance part="P+2" gate="1" x="223.52" y="93.98"/>
 </instances>
 <busses>
@@
 <net name="GND" class="1">
 <segment>
-<wire x1="139.7" y1="170.18" x2="139.7" y2="142.24" width="0.1524" layer="91"/>
 <pinref part="GND15" gate="1" pin="GND"/>
-<pinref part="GND14" gate="1" pin="P"/>
-<wire x1="139.7" y1="142.24" x2="139.7" y2="134.62" width="0.1524" layer="91"/>
+<wire x1="149.86" y1="142.24" x2="149.86" y2="134.62" width="0.1524" layer="91"/>
 <wire x1="149.86" y1="144.78" x2="149.86" y2="142.24" width="0.1524" layer="91"/>
-<wire x1="149.86" y1="142.24" x2="139.7" y2="142.24" width="0.1524" layer="91"/>
 <wire x1="154.94" y1="144.78" x2="154.94" y2="142.24" width="0.1524" layer="91"/>
 <wire x1="154.94" y1="142.24" x2="149.86" y2="142.24" width="0.1524" layer="91"/>
 <junction x="149.86" y="142.24"/>
-<junction x="139.7" y="142.24"/>
 <pinref part="R78" gate="G$1" pin="1"/>
 <pinref part="R79" gate="G$1" pin="1"/>
@@
 </segment>
 </net>
-<net name="+12V" class="0">
-<segment>
-<pinref part="P+7" gate="1" pin="+12V"/>
-<pinref part="U$37" gate="G$1" pin="VDD"/>
-<wire x1="228.6" y1="63.5" x2="223.52" y2="63.5" width="0.1524" layer="91"/>
-<wire x1="223.52" y1="63.5" x2="223.52" y2="78.74" width="0.1524" layer="91"/>
-<pinref part="R88" gate="G$1" pin="2"/>
-<wire x1="223.52" y1="78.74" x2="223.52" y2="91.44" width="0.1524" layer="91"/>
-<wire x1="231.14" y1="78.74" x2="223.52" y2="78.74" width="0.1524" layer="91"/>
-<junction x="223.52" y="78.74"/>
-</segment>
-</net>
 <net name="CHARGE_PWM" class="0">
 <segment>
@@
 </segment>
 </net>
+<net name="+15V" class="0">
+<segment>
+<pinref part="U$37" gate="G$1" pin="VDD"/>
+<wire x1="228.6" y1="63.5" x2="223.52" y2="63.5" width="0.1524" layer="91"/>
+<wire x1="223.52" y1="63.5" x2="223.52" y2="78.74" width="0.1524" layer="91"/>
+<pinref part="R88" gate="G$1" pin="2"/>
+<wire x1="223.52" y1="78.74" x2="223.52" y2="91.44" width="0.1524" layer="91"/>
+<wire x1="231.14" y1="78.74" x2="223.52" y2="78.74" width="0.1524" layer="91"/>
+<junction x="223.52" y="78.74"/>
+<pinref part="P+2" gate="1" pin="+15V"/>
+</segment>
+</net>
 </nets>
 </sheet>
@@
 <instance part="FRAME3" gate="G$1" x="0" y="0"/>
 <instance part="U$1" gate="A" x="91.44" y="132.08"/>
-<instance part="P+11" gate="VCC" x="63.5" y="149.86"/>
 <instance part="C1" gate="G$1" x="86.36" y="127" rot="R90"/>
 <instance part="C14" gate="G$1" x="55.88" y="129.54" rot="R90"/>
@@
 </segment>
 </net>
-<net name="VCC" class="0">
-<segment>
-<pinref part="U$1" gate="A" pin="VIN"/>
-<wire x1="93.98" y1="129.54" x2="63.5" y2="129.54" width="0.1524" layer="91"/>
-<wire x1="63.5" y1="129.54" x2="63.5" y2="147.32" width="0.1524" layer="91"/>
-<pinref part="P+11" gate="VCC" pin="VCC"/>
-<pinref part="C14" gate="G$1" pin="2"/>
-<wire x1="60.96" y1="129.54" x2="63.5" y2="129.54" width="0.1524" layer="91"/>
-<junction x="63.5" y="129.54"/>
-</segment>
-</net>
 <net name="N$1" class="0">
 <segment>
@@
 </segment>
 </net>
+<net name="BATTERY+" class="0">
+<segment>
+<pinref part="U$1" gate="A" pin="VIN"/>
+<wire x1="93.98" y1="129.54" x2="63.5" y2="129.54" width="0.1524" layer="91"/>
+<wire x1="63.5" y1="129.54" x2="63.5" y2="147.32" width="0.1524" layer="91"/>
+<pinref part="C14" gate="G$1" pin="2"/>
+<wire x1="60.96" y1="129.54" x2="63.5" y2="129.54" width="0.1524" layer="91"/>
+<junction x="63.5" y="129.54"/>
+<label x="63.5" y="147.32" size="1.778" layer="95" rot="R180" xref="yes"/>
+</segment>
+</net>

Commit message: backup
Parts:
- removed R73: (no value), rcl:R-EU_R0603
Connections:
- removed net N$57: R73.2, U$36.G
- net EN_LED: now also U$36.G; no longer R73.1
Changed lines of the file:
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@@
 <part name="U$36" library="BM_pre" deviceset="SI4490" device=""/>
 <part name="GND29" library="supply1" deviceset="GND" device=""/>
-<part name="R73" library="rcl" deviceset="R-EU_" device="R0603"/>
 <part name="R74" library="rcl" deviceset="R-EU_" device="R0603" value="0"/>
 <part name="R75" library="rcl" deviceset="R-EU_" device="R0603" value="0"/>
@@
 <instance part="U$36" gate="G$1" x="139.7" y="63.5" rot="MR0"/>
 <instance part="GND29" gate="1" x="137.16" y="53.34"/>
-<instance part="R73" gate="G$1" x="160.02" y="60.96" rot="R180"/>
 <instance part="15V" gate="1" x="68.58" y="99.06"/>
 </instances>
@@
 </segment>
 </net>
-<net name="N$57" class="0">
-<segment>
+<net name="EN_LED" class="0">
+<segment>
+<label x="177.8" y="60.96" size="1.778" layer="95" xref="yes"/>
 <pinref part="U$36" gate="G$1" pin="G"/>
-<pinref part="R73" gate="G$1" pin="2"/>
-<wire x1="142.24" y1="60.96" x2="154.94" y2="60.96" width="0.1524" layer="91"/>
-</segment>
-</net>
-<net name="EN_LED" class="0">
-<segment>
-<pinref part="R73" gate="G$1" pin="1"/>
-<wire x1="165.1" y1="60.96" x2="177.8" y2="60.96" width="0.1524" layer="91"/>
-<label x="177.8" y="60.96" size="1.778" layer="95" xref="yes"/>
-</segment>
-</net>
+<wire x1="142.24" y1="60.96" x2="177.8" y2="60.96" width="0.1524" layer="91"/>
+</segment>
+</net>

Commit message: bm style
Other:
- moved on the sheet: C11, C12, C3, C9, CELL1, CELL2, CELL3, CELL4, CELL5, CELL6, PAD1, PAD2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
