File: MotorControl/v0.2/skatemate_proto.brd (EAGLE design)
At the start: 72.1 x 91.1 mm, 100 parts, among them IC1 REG1117, U1 DRV8301DCAR, U2 STM32F303XD/XELQFP64, U3 RFM75, X1 ABM3B

Commit message: Added missing values
Parts:
- C1, C6: value (none) -> 2n2
- C23: value (none) -> 22n
- R1, R2, R4, R5, R7, R8: value (none) -> 10
- R3, R6: value R_EU -> 1m
Changed lines of the file:
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@@
 </autorouter>
 <elements>
-<element name="C1" library="skatemate" package="C0805" value="" x="34.036" y="46.482" rot="MR90"/>
+<element name="C1" library="skatemate" package="C0805" value="2n2" x="34.036" y="46.482" rot="MR90"/>
 <element name="C14" library="skatemate" package="C0805" value="10n" x="28.194" y="61.976" rot="R270"/>
 <element name="C22" library="skatemate" package="C0805" value="100n" x="40.894" y="58.166" rot="R90"/>
@@
 <element name="C18" library="skatemate" package="C1206" value="4u7" x="32.004" y="62.738" rot="R270"/>
 <element name="C15" library="skatemate" package="C0805" value="100n" x="34.29" y="61.976" rot="R270"/>
-<element name="C6" library="skatemate" package="C0805" value="" x="36.576" y="43.18"/>
+<element name="C6" library="skatemate" package="C0805" value="2n2" x="36.576" y="43.18"/>
 <element name="C12" library="skatemate" package="C1206" value="4u7" x="32.766" y="42.418" rot="R90"/>
 <element name="C11" library="skatemate" package="C0805" value="100n" x="33.782" y="38.862"/>
@@
 <element name="C3" library="skatemate" package="C1206" value="2u2" x="44.958" y="35.56" rot="MR180"/>
 <element name="C4" library="skatemate" package="C1206" value="2u2" x="44.958" y="33.02" rot="MR180"/>
-<element name="C23" library="skatemate" package="C0805" value="" x="14.478" y="48.26" rot="R270"/>
+<element name="C23" library="skatemate" package="C0805" value="22n" x="14.478" y="48.26" rot="R270"/>
 <element name="D7" library="skatemate" package="SOD80C" value="BAS85" x="30.988" y="18.034"/>
 <element name="D8" library="skatemate" package="SOD80C" value="BAS85" x="30.988" y="14.478"/>
@@
 </element>
 <element name="L1" library="skatemate" package="SDR0805" value="" x="29.464" y="76.2" rot="R270"/>
-<element name="R1" library="skatemate" package="R0805" value="" x="58.674" y="82.804" rot="MR180"/>
+<element name="R1" library="skatemate" package="R0805" value="10" x="58.674" y="82.804" rot="MR180"/>
 <element name="R12" library="skatemate" package="R0805" value="2k2" x="56.388" y="52.07" rot="R180"/>
 <element name="R13" library="skatemate" package="R0805" value="39k" x="56.642" y="22.86"/>
@@
 <element name="R23" library="skatemate" package="R0805" value="18k" x="9.652" y="41.656" rot="MR0"/>
 <element name="R24" library="skatemate" package="R0805" value="18k" x="9.652" y="45.72" rot="MR0"/>
-<element name="R2" library="skatemate" package="R0805" value="" x="54.356" y="58.928" rot="MR180"/>
-<element name="R4" library="skatemate" package="R0805" value="" x="60.198" y="56.896" rot="MR180"/>
-<element name="R5" library="skatemate" package="R0805" value="" x="52.832" y="33.274" rot="MR180"/>
-<element name="R7" library="skatemate" package="R0805" value="" x="58.166" y="31.496" rot="MR180"/>
-<element name="R8" library="skatemate" package="R0805" value="" x="49.022" y="9.144" rot="MR180"/>
+<element name="R2" library="skatemate" package="R0805" value="10" x="54.356" y="58.928" rot="MR180"/>
+<element name="R4" library="skatemate" package="R0805" value="10" x="60.198" y="56.896" rot="MR180"/>
+<element name="R5" library="skatemate" package="R0805" value="10" x="52.832" y="33.274" rot="MR180"/>
+<element name="R7" library="skatemate" package="R0805" value="10" x="58.166" y="31.496" rot="MR180"/>
+<element name="R8" library="skatemate" package="R0805" value="10" x="49.022" y="9.144" rot="MR180"/>
 <element name="R9" library="skatemate" package="R0805" value="39k" x="58.42" y="71.12"/>
 <element name="R10" library="skatemate" package="R0805" value="2k2" x="57.658" y="66.04" rot="R180"/>
 <element name="R11" library="skatemate" package="R0805" value="39k" x="56.388" y="48.006"/>
-<element name="R3" library="skatemate" package="R2512" value="R_EU" x="46.736" y="66.548" rot="MR270"/>
-<element name="R6" library="skatemate" package="R2512" value="R_EU" x="46.736" y="41.148" rot="MR270"/>
+<element name="R3" library="skatemate" package="R2512" value="1m" x="46.736" y="66.548" rot="MR270"/>
+<element name="R6" library="skatemate" package="R2512" value="1m" x="46.736" y="41.148" rot="MR270"/>
 <element name="U1" library="skatemate" package="SOP50P810X120-57N" value="DRV8301DCAR" x="29.718" y="52.324">
 <attribute name="PACKAGE" value="HTSSOP-56" x="29.718" y="52.324" size="1.778" layer="27" display="off"/>
